Commit message: feat(hardware): regenerate stack and link architecture docs

File: description/ros2_control/inmoov_ros2_control.xacro (robot description, xacro)
@@ -14,6 +14,96 @@
       </xacro:unless>
     </hardware>
+      <joint name="i01.leftHand.thumb_link_joint">
+          <param name="virtual_pin">0</param>
+          <param name="servo_type">300</param>
+          <param name="offset_rad">0</param>
+          <param name="direction">1</param>
+          <param name="scale">1</param>
+          <param name="servo_min_rad">0</param>
+          <param name="servo_max_rad">3.14159</param>
+          <param name="servo_default_rad">0</param>
+          <command_interface name="position">
+            <param name="min">0.0</param>
+            <param name="max">1.5708</param>
+          </command_interface>
+          <state_interface name="position" />
+      </joint>
+      <joint name="i01.leftHand.index_link_joint">
+          <param name="virtual_pin">1</param>
+          <param name="servo_type">300</param>
+          <param name="offset_rad">0</param>
+          <param name="direction">1</param>
+          <param name="scale">1</param>
+          <param name="servo_min_rad">0</param>
+          <param name="servo_max_rad">3.14159</param>
+          <param name="servo_default_rad">0</param>
+          <command_interface name="position">
+            <param name="min">0.0</param>
+            <param name="max">1.5708</param>
+          </command_interface>
+          <state_interface name="position" />
+      </joint>
+      <joint name="i01.leftHand.majeure_link_joint">
+          <param name="virtual_pin">2</param>
+          <param name="servo_type">300</param>
+          <param name="offset_rad">0</param>
+          <param name="direction">1</param>
+          <param name="scale">1</param>
+          <param name="servo_min_rad">0</param>
+          <param name="servo_max_rad">3.14159</param>
+          <param name="servo_default_rad">0</param>
+          <command_interface name="position">
+            <param name="min">0.0</param>
+            <param name="max">1.5708</param>
+          </command_interface>
+          <state_interface name="position" />
+      </joint>
+      <joint name="i01.leftHand.ringFinger_link_joint">
+          <param name="virtual_pin">3</param>
+          <param name="servo_type">300</param>
+          <param name="offset_rad">0</param>
+          <param name="direction">1</param>
+          <param name="scale">1</param>
+          <param name="servo_min_rad">0</param>
+          <param name="servo_max_rad">3.14159</param>
+          <param name="servo_default_rad">0</param>
+          <command_interface name="position">
+            <param name="min">0.0</param>
+            <param name="max">1.5708</param>
+          </command_interface>
+          <state_interface name="position" />
+      </joint>
+      <joint name="i01.leftHand.pinky_link_joint">
+          <param name="virtual_pin">4</param>
+          <param name="servo_type">300</param>
+          <param name="offset_rad">0</param>
+          <param name="direction">1</param>
+          <param name="scale">1</param>
+          <param name="servo_min_rad">0</param>
+          <param name="servo_max_rad">3.141592653589793</param>
+          <param name="servo_default_rad">0</param>
+          <command_interface name="position">
+            <param name="min">0.0</param>
+            <param name="max">1.5708</param>
+          </command_interface>
+          <state_interface name="position" />
+      </joint>
+      <joint name="left_wrist_z_link_joint">
+          <param name="virtual_pin">5</param>
+          <param name="servo_type">300</param>
+          <param name="offset_rad">2.61799</param>
+          <param name="direction">1</param>
+          <param name="scale">1</param>
+          <param name="servo_min_rad">0</param>
+          <param name="servo_max_rad">5.23599</param>
+          <param name="servo_default_rad">0</param>
+          <command_interface name="position">
+            <param name="min">-1.5708</param>
+            <param name="max">1.5708</param>
+          </command_interface>
+          <state_interface name="position" />
+      </joint>
       <joint name="left_shoulder_z_link_joint">
-          <param name="virtual_pin">0</param>
+          <param name="virtual_pin">6</param>
           <param name="servo_type">270</param>
           <param name="offset_rad">1.5708</param>
@@ -30,5 +120,5 @@
       </joint>
       <joint name="left_shoulder_x_link_joint">
-          <param name="virtual_pin">1</param>
+          <param name="virtual_pin">7</param>
           <param name="servo_type">270</param>
           <param name="offset_rad">0</param>
@@ -45,99 +135,9 @@
       </joint>
       <joint name="left_elbow_x_link_joint">
-          <param name="virtual_pin">2</param>
-          <param name="servo_type">270</param>
-          <param name="offset_rad">0</param>
-          <param name="direction">1</param>
-          <param name="scale">1</param>
-          <param name="servo_min_rad">0</param>
-          <param name="servo_max_rad">3.14159</param>
-          <param name="servo_default_rad">0</param>
-          <command_interface name="position">
-            <param name="min">0.0</param>
-            <param name="max">1.5708</param>
-          </command_interface>
-          <state_interface name="position" />
-      </joint>
-      <joint name="left_wrist_z_link_joint">
-          <param name="virtual_pin">3</param>
-          <param name="servo_type">300</param>
-          <param name="offset_rad">2.61799</param>
-          <param name="direction">1</param>
-          <param name="scale">1</param>
-          <param name="servo_min_rad">0</param>
-          <param name="servo_max_rad">5.23599</param>
-          <param name="servo_default_rad">2.61799</param>
-          <command_interface name="position">
-            <param name="min">-1.5708</param>
-            <param name="max">1.5708</param>
-          </command_interface>
-          <state_interface name="position" />
-      </joint>
-      <joint name="i01.leftHand.thumb_link_joint">
-          <param name="virtual_pin">4</param>
-          <param name="servo_type">300</param>
-          <param name="offset_rad">0</param>
-          <param name="direction">1</param>
-          <param name="scale">1</param>
-          <param name="servo_min_rad">0</param>
-          <param name="servo_max_rad">3.14159</param>
-          <param name="servo_default_rad">0</param>
-          <command_interface name="position">
-            <param name="min">0.0</param>
-            <param name="max">1.5708</param>
-          </command_interface>
-          <state_interface name="position" />
-      </joint>
-      <joint name="i01.leftHand.index_link_joint">
-          <param name="virtual_pin">5</param>
-          <param name="servo_type">300</param>
-          <param name="offset_rad">0</param>
-          <param name="direction">1</param>
-          <param name="scale">1</param>
-          <param name="servo_min_rad">0</param>
-          <param name="servo_max_rad">3.14159</param>
-          <param name="servo_default_rad">0</param>
-          <command_interface name="position">
-            <param name="min">0.0</param>
-            <param name="max">1.5708</param>
-          </command_interface>
-          <state_interface name="position" />
-      </joint>
-      <joint name="i01.leftHand.majeure_link_joint">
-          <param name="virtual_pin">6</param>
-          <param name="servo_type">300</param>
-          <param name="offset_rad">0</param>
-          <param name="direction">1</param>
-          <param name="scale">1</param>
-          <param name="servo_min_rad">0</param>
-          <param name="servo_max_rad">3.14159</param>
-          <param name="servo_default_rad">0</param>
-          <command_interface name="position">
-            <param name="min">0.0</param>
-            <param name="max">1.5708</param>
-          </command_interface>
-          <state_interface name="position" />
-      </joint>
-      <joint name="i01.leftHand.ringFinger_link_joint">
-          <param name="virtual_pin">7</param>
-          <param name="servo_type">300</param>
-          <param name="offset_rad">0</param>
-          <param name="direction">1</param>
-          <param name="scale">1</param>
-          <param name="servo_min_rad">0</param>
-          <param name="servo_max_rad">3.14159</param>
-          <param name="servo_default_rad">0</param>
-          <command_interface name="position">
-            <param name="min">0.0</param>
-            <param name="max">1.5708</param>
-          </command_interface>
-          <state_interface name="position" />
-      </joint>
-      <joint name="i01.leftHand.pinky_link_joint">
           <param name="virtual_pin">8</param>
-          <param name="servo_type">300</param>
-          <param name="offset_rad">0</param>
-          <param name="direction">1</param>
-          <param name="scale">0.25</param>
+          <param name="servo_type">270</param>
+          <param name="offset_rad">0</param>
+          <param name="direction">1</param>
+          <param name="scale">1</param>
           <param name="servo_min_rad">0</param>
           <param name="servo_max_rad">3.14159</param>
